File: joy2ps2/avillena/SNES-GamePad.brd (EAGLE design)
At the start: 142.4 x 49.3 mm, 15 parts

Commit message: Hago commit de lo último
Parts:
- removed E$1: (no value), pinhead:2X06
- removed E$2, E$3: (no value), pinhead:1X02
- added A1: ANTENA, ,giltesa:ANTENA-AIROHA
- added BATTERY: VCC 3.7V, ,giltesa:1X02_SMD_BIG
- added BTN-0: L, ,giltesa:1X02_SMD
- added BTN-1: R, ,giltesa:1X02_SMD
- added BTN-RST: CONNECT, ,giltesa:SWITCH-90º
- added C10, C11, C12, C19, C2, C20, C22, C26, C3, C32, C4, C5, C6, L3, L4, L5, L6: C0603, ,giltesa:C0603
- added E2: C0805, ,giltesa:C0805
- added L1: C1206, ,giltesa:C1206
- added LBLUE, LGREEN, LRED: (no value), led:CHIPLED_0805
- added R1, R2, R3, R4, R5, R6, R7, R8: 22kΩ, ,giltesa:R0603
- added R10, R11: 2.2kΩ, ,giltesa:R0603
- added R12, R15: 330Ω, ,giltesa:R0603
- added R13: 10Ω, ,giltesa:R0603
- added R16: 10kΩ, ,giltesa:R0603
- added R17, R9: 4.7kΩ, ,giltesa:R0603
- added R18: 1kΩ, ,giltesa:R0603
- added S2: INTERRUPTOR_1, ,giltesa:INTERRUPTOR_1
- added SJ1, SJ2, SJ3: JUMPER-SMD, ,giltesa:JUMPER-SMD
- added U$1: (no value), ,ppp:SNES-LOGO
- added U1: AIROHA AB1108, ,giltesa:QFN56_6MM
- added U2: EEPROM1, ,giltesa:TSSOP8
- added U2': EEPROM2, ,giltesa:M8-EEPROM
- added U3: SOT23-5, ,giltesa:SOT23-5
- added USB: MICRO_USB_1, ,giltesa:MICRO_USB_1
- added Y1: CRISTAL, ,giltesa:CRISTAL-SMD-3X2.5MM
Connections:
- removed net S$1: BTN-2.1, BTN-3.2, BTN-4.1, BTN-5.2, BTN-6.2, BTN-7.2, BTN-8.1, BTN-9.1, BTN-DEL.1, BTN-ENTER.1, E$1.11, E$2.1, E$3.2
- new net 3.7V: BATTERY.VCC, C6.1, E2.1, S2.VCCIN, U3.1
- new net 5V: C2.1, R15.2, R16.2, U3.5, USB.VCC
- new net BAT: C10.1, C12.1, C32.2, R1.1, R10.1, R11.1, R12.1, R18.2, R2.1, R3.1, R4.1, R5.2, R6.2, R7.2, R8.2, R9.1, S2.VCCOUT, U1.P10, U1.P11, U1.P16, U1.P19, U2'.8, U2.8
- new net COL1: BTN-1.1, BTN-DEL.2, U1.P38
- new net COL2: BTN-2.2, U1.P37
- new net COL3: BTN-3.1, U1.P36
- new net COL4: BTN-4.1, BTN-ENTER.1, U1.P35
- new net COL5: BTN-0.1, BTN-5.2, U1.P34
- new net COL6: BTN-6.2, BTN-8.2, BTN-9.2, U1.P33
- new net COL7: BTN-7.2, U1.P32
- new net CONNECT: BTN-RST.1, U1.P48
- new net FIL1: BTN-1.2, BTN-2.1, BTN-3.2, BTN-4.2, BTN-5.1, BTN-6.1, BTN-7.1, R8.1, U1.P47
- new net FIL2: BTN-8.1, BTN-DEL.1, R2.2, U1.P6
- new net FIL3: BTN-0.2, BTN-9.1, R3.2, U1.P24
- new net FIL4: BTN-ENTER.2, R4.2, U1.P25
- new net GND: A1.GND, BATTERY.GND, BTN-RST.2, BTN-RST.GND1, BTN-RST.GND2, C10.2, C11.1, C12.2, C2.2, C20.1, C22.1, C26.2, C3.2, C32.1, C4.1, C5.1, C6.2, E2.2, L4.1, LGREEN.C, R17.2, S2.GND1, S2.GND2, U1.P0, U1.P13, U2'.1, U2'.2, U2'.3, U2'.4, U2.1, U2.2, U2.3, U2.4, U3.2, USB.GND0, USB.GND1, USB.GND2, Y1.GND1, Y1.GND2
- new net N$1: LRED.A, R15.1
- new net N$2: C22.2, L5.2, U1.P50
- new net N$3: SJ1.2, USB.OTG
- new net N$35: LBLUE.C, U1.P28
- new net N$36: LRED.C, R16.1, U3.3
- new net N$37: R17.1, U3.4
- new net N$39: LBLUE.A, R12.2
- new net N$4: LGREEN.A, R18.1
- new net N$40: C26.1, R13.1, U1.P43
- new net N$45: C11.2, C20.2, C3.1, L1.2, L5.1, L6.1, R13.2, U1.P3, U1.P42, U1.P52, U1.P53, U1.P9
- new net N$46: R1.2, U1.P18
- new net N$48: R5.1, U1.P44
- new net N$49: R6.1, U1.P45
- new net N$5: C19.1, L3.2, L4.2
- new net N$50: R7.1, U1.P46
- new net N$52: L1.1, U1.P12
- new net N$6: A1.SIGNAL, L3.1
- new net N$7: C19.2, L6.2, U1.P51
- new net N$8: SJ3.2, USB.D-
- new net N$9: SJ2.2, USB.D+
- new net RX: SJ3.1, U1.P23
- new net SCL: R10.2, U1.P30, U2'.6, U2.6
- new net SDA: R11.2, U1.P31, U2'.5, U2.5
- new net TX: SJ2.1, U1.P22
- new net WP: R9.2, SJ1.1, U1.P29, U2'.7, U2.7
- new net X1: C5.2, U1.P1, Y1.P2
- new net X2: C4.2, U1.P2, Y1.P1
Routing:
- net COL6: track 0.00 -> 140.6 mm, vias 0 -> 5
- net FIL3: track 0.00 -> 138.6 mm, vias 0 -> 2
- net BAT: track 0.00 -> 137.2 mm, vias 0 -> 4
- net FIL1: track 0.00 -> 132.5 mm, vias 0 -> 3
- net COL5: track 0.00 -> 110.2 mm, vias 0 -> 4
- net COL4: track 0.00 -> 106.2 mm, vias 0 -> 3
- net COL2: track 0.00 -> 102.2 mm, vias 0 -> 3
- net COL1: track 0.00 -> 93.9 mm, vias 0 -> 4
- net WP: track 0.00 -> 87.4 mm, vias 0 -> 4
- net 3.7V: track 0.00 -> 86.5 mm, vias 0 -> 3
- net FIL2: track 0.00 -> 83.6 mm, vias 0 -> 7
- net N$35: track 0.00 -> 83.5 mm, vias 0 -> 3
- net RX: track 0.00 -> 81.7 mm, vias 0 -> 4
- net TX: track 0.00 -> 78.2 mm, vias 0 -> 4
- net N$45: track 0.00 -> 53.9 mm
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- added copper zone on layer 1, net GND
- added copper zone on layer 16, net GND
Other:
- board text added: "Battery 3.7V"
- board text added: "Blue"
- board text added: "GND"
- board text added: "Green"
- board text added: "OFF - ON"
- board text added: "RX"
- board text added: "Red"
- board text added: "TX"
- board text added: "USB"
- board text added: "VCC"
- board text added: "WP"
- board text added: "Y"
