File: joy2ps2/avillena/Arduino Nano-Rev3.2.brd (EAGLE design)
At the start: 128.4 x 40.5 mm, 22 parts, among them IC3 ATMEGA328P-AU, Y1 16MHz

Commit message: Fallo arreglado
Routing:
- net GND: track 284.2 -> 294.8 mm
- net D8: track 32.5 -> 34.3 mm
- net D4: track 80.9 -> 82.6 mm
- net D6: track 50.4 -> 51.5 mm
- net D11/MOSI: track 142.5 -> 143.5 mm
Changed lines of the file:
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@@
 <wire x1="56.092225" y1="18.161" x2="54.7415375" y2="16.8103125" width="0.254" layer="1"/>
 <wire x1="21.209" y1="6.604" x2="36.322" y2="6.604" width="0.254" layer="16"/>
-<wire x1="36.322" y1="6.604" x2="54.229" y2="24.511" width="0.254" layer="16"/>
-<wire x1="54.229" y1="24.511" x2="57.531" y2="24.511" width="0.254" layer="16"/>
-<wire x1="57.531" y1="24.511" x2="59.563" y2="26.543" width="0.254" layer="16"/>
+<wire x1="36.322" y1="6.604" x2="55.753" y2="26.035" width="0.254" layer="16"/>
+<wire x1="57.531" y1="24.511" x2="59.563" y2="26.543" width="0" layer="19" extent="1-16"/>
+<wire x1="55.753" y1="26.035" x2="55.753" y2="27.178" width="0.254" layer="16"/>
+<wire x1="55.753" y1="27.178" x2="56.388" y2="27.813" width="0.254" layer="16"/>
+<wire x1="59.563" y1="26.543" x2="59.055" y2="26.543" width="0.254" layer="16"/>
+<wire x1="59.055" y1="26.543" x2="57.785" y2="27.813" width="0.254" layer="16"/>
+<wire x1="57.785" y1="27.813" x2="56.388" y2="27.813" width="0.254" layer="16"/>
 </signal>
 <signal name="D3">
@@
 <wire x1="48.133" y1="20.574" x2="48.133" y2="20.176621875" width="0.254" layer="1"/>
 <wire x1="48.133" y1="20.176621875" x2="48.670884375" y2="19.6387375" width="0.254" layer="1"/>
-<wire x1="22.352" y1="35.814" x2="47.752" y2="35.814" width="0.254" layer="16"/>
-<wire x1="47.752" y1="35.814" x2="54.483" y2="29.083" width="0.254" layer="16"/>
 <wire x1="21.2259" y1="34.6879" x2="22.352" y2="35.814" width="0.254" layer="16"/>
+<wire x1="54.483" y1="29.083" x2="53.213" y2="27.813" width="0.254" layer="16"/>
+<wire x1="53.213" y1="27.813" x2="48.387" y2="27.813" width="0.254" layer="16"/>
+<wire x1="48.387" y1="27.813" x2="40.386" y2="35.814" width="0.254" layer="16"/>
+<wire x1="40.386" y1="35.814" x2="22.352" y2="35.814" width="0.254" layer="16"/>
 </signal>
 <signal name="D7">
@@
 <contactref element="JP1" pad="4"/>
 <wire x1="59.0719" y1="18.2299" x2="59.0719" y2="23.3849" width="0.254" layer="16"/>
-<wire x1="53.213" y1="27.813" x2="60.198" y2="27.813" width="0.254" layer="16"/>
 <wire x1="60.198" y1="27.813" x2="60.833" y2="27.178" width="0.254" layer="16"/>
 <wire x1="60.833" y1="27.178" x2="60.833" y2="25.146" width="0.254" layer="16"/>
@@
 <wire x1="46.609" y1="21.082" x2="46.609" y2="19.437884375" width="0.254" layer="1"/>
 <wire x1="46.609" y1="19.437884375" x2="47.539515625" y2="18.50736875" width="0.254" layer="1"/>
-<wire x1="53.213" y1="27.813" x2="51.943" y2="29.083" width="0.254" layer="16"/>
+<wire x1="60.198" y1="27.813" x2="58.928" y2="27.813" width="0.254" layer="16"/>
+<wire x1="58.928" y1="27.813" x2="58.293" y2="28.448" width="0.254" layer="16"/>
+<wire x1="58.293" y1="28.448" x2="58.293" y2="29.718" width="0.254" layer="16"/>
+<wire x1="58.293" y1="29.718" x2="57.658" y2="30.353" width="0.254" layer="16"/>
+<wire x1="57.658" y1="30.353" x2="53.213" y2="30.353" width="0.254" layer="16"/>
+<wire x1="53.213" y1="30.353" x2="51.943" y2="29.083" width="0.254" layer="16"/>
 </signal>
 <signal name="D9">
@@
 <wire x1="40.838" y1="33.508" x2="40.838" y2="17.582" width="0.254" layer="1"/>
 <wire x1="40.838" y1="17.582" x2="40.894" y2="17.526" width="0.254" layer="1"/>
-<wire x1="59.563" y1="29.083" x2="52.324" y2="36.322" width="0.254" layer="16"/>
-<wire x1="52.324" y1="36.322" x2="17.78" y2="36.322" width="0.254" layer="16"/>
+<wire x1="54.102" y1="36.322" x2="17.78" y2="36.322" width="0.254" layer="16"/>
 <wire x1="17.78" y1="36.322" x2="7.493" y2="26.035" width="0.254" layer="16"/>
 <wire x1="7.493" y1="26.035" x2="7.493" y2="19.431" width="0.254" layer="16"/>
 <wire x1="7.493" y1="19.431" x2="24.638" y2="2.286" width="0.254" layer="16"/>
 <wire x1="24.638" y1="2.286" x2="33.655" y2="2.286" width="0.254" layer="16"/>
+<wire x1="54.102" y1="36.322" x2="59.563" y2="30.861" width="0.254" layer="16"/>
+<wire x1="59.563" y1="30.861" x2="59.563" y2="29.083" width="0.254" layer="16"/>
 </signal>
 <signal name="D12/MISO">
@@
 <vertex x="1.778" y="0.889"/>
 </polygon>
-<wire x1="59.07355" y1="17.07585" x2="58.6994" y2="21.4122" width="0" layer="19" extent="1-16"/>
+<wire x1="59.07355" y1="17.07585" x2="58.74315" y2="17.07585" width="0.4064" layer="16"/>
+<wire x1="58.74315" y1="17.07585" x2="57.023" y2="18.796" width="0.4064" layer="16"/>
+<wire x1="57.023" y1="18.796" x2="57.023" y2="26.543" width="0.4064" layer="16"/>
 </signal>
 </signals>
