File: ZXUnoCompanion-2/ZXUno_Companion_2.brd (EAGLE design)
At the start: 240 x 155 mm, 44 parts, among them Q1 2N3904, Q2 2N3904, Q3 2N3904, Q4 2N3904, U1 ARDUINO_MEGA_R3FULL, X1 TOBU3, X2 TOBU3, X3 DB15

Commit message: Update 2
Parts:
- removed B1: MEGA2560_COREFULL, spark2k06:MEGA2560_CORE
- removed JOYSTICK1, JOYSTICK2: (no value), SparkFun-Connectors:DB9_MALE
- removed JP1: (no value), pinhead:1X11
- removed JP2: (no value), pinhead:1X13
- removed JP3: (no value), pinhead:1X03
- removed PWCON_ZXUNO: (no value), pinhead:1X04
- removed U1: ARDUINO_MEGA_R3FULL, SparkFun-Boards:ARDUINO_MEGA
- added ARDUINO_MEGA: ARDUINO_MEGA_R3FULL, SparkFun-Boards2:ARDUINO_MEGA
- added ATMEGA128: MEGA128-A, atmel:TQFP64
- added EXTRASW: PS-22F03, A03 PS-22F03:PS-22F03
- added EXTRASW_CFG, INTERNAL_SPEAKERS, VIDEO_CFG: (no value), pinhead:1X03
- added ICSP: AVR_SPI_PRG_6NS, SparkFun-Connectors:2X3-NS
- added JOYSTICK_1, JOYSTICK_2: (no value), SparkFun-Connectors:DB9_MALE
- added JOYZXUNO_CFG: (no value), pinhead:2X09
- added KB1: (no value), pinhead:1X13
- added KB2: (no value), pinhead:1X11
- added KB_BIDIR: PC817, optocoupler:DIL04
- added PW_CONTROL: IRLML6344TRPBF, International_Rectifier_By_element14_Batch_1:SOT95P240X112-3N
- added PW_SWITCH: (no value), pinhead:1X02
- added R7: 220R, resistor:0204/7
- added SDCARD: (no value), zxuno_rev_mcleod:SDCMF-10915W010
- added SDCARD_ZXUNO: (no value), pinhead:1X06
- added TAPE: 22-23-2051, con-molex:22-23-2051
- added U$1: MICRO-USB-B, micro usb B - 4LEGS:MICRO_USB_4_LEGS
- added USB_ARDUINO: (no value), pinhead:1X05
- added X5: (no value), con-subd-spark2k06:F09D
- R1, R2, R3, R4, R5, R6: device resistor:0207/10 -> resistor:0204/7
- TZXDUINO: device pinhead:2X04 -> pinhead:2X05
- moved R6 114.9 mm to (86.0, 61.1)
- moved Q3 114.6 mm to (79.3, 59.9), turned to 180 degrees
- moved C3 113.9 mm to (79.3, 66.4), turned to 180 degrees
- moved Q4 101.2 mm to (79.6, 51.1), turned to 180 degrees
- moved R5 100.2 mm to (72.2, 61.1)
- moved TZXDUINO 88.0 mm to (31.2, 74.5), turned to 0 degrees
- moved R4 79.2 mm to (37.8, 56.3)
- moved Q2 78.4 mm to (30.9, 54.8), turned to 180 degrees
- moved C2 77.9 mm to (30.9, 61.2), turned to 180 degrees
- moved R1 72.5 mm to (17.8, 56.8), turned to 270 degrees
- moved Q1 72.2 mm to (10.6, 55.1), turned to 180 degrees
- moved C1 71.7 mm to (10.6, 61.9), turned to 180 degrees
- moved R3 64.5 mm to (23.8, 56.3)
- moved R2 59.0 mm to (3.34, 57.0)
- moved X4 38.2 mm to (-40.7, 79.0)
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Connections:
- removed net SW1: PWCON_ZXUNO.3
- removed net SW2: PWCON_ZXUNO.4
- new net CS1: SDCARD.1, SDCARD_ZXUNO.1
- new net D+: U$1.D+, USB_ARDUINO.3
- new net D-: U$1.D-, USB_ARDUINO.4
- new net EXTRA: ARDUINO_MEGA.52, ATMEGA128.45, EXTRASW_CFG.1
- new net GND_POW: ARDUINO_MEGA.GND@0, ARDUINO_MEGA.GND@1, ARDUINO_MEGA.GND@4, ATMEGA128.22, ATMEGA128.53, ATMEGA128.63, EXTRASW.5, EXTRASW.6, ICSP.6, KB_BIDIR.2, PW_CONTROL.3, PW_SWITCH.1, U$1.GND, USB_ARDUINO.1
- new net ID: U$1.ID, USB_ARDUINO.2
- new net JOYZXUNO_1': ARDUINO_MEGA.A7, ATMEGA128.57, JOYZXUNO_CFG.1
- new net JOYZXUNO_2': ARDUINO_MEGA.A8, ATMEGA128.56, JOYZXUNO_CFG.3
- new net JOYZXUNO_3': ARDUINO_MEGA.A9, ATMEGA128.55, JOYZXUNO_CFG.5
- new net JOYZXUNO_4': ARDUINO_MEGA.A10, ATMEGA128.54, JOYZXUNO_CFG.7
- new net JOYZXUNO_5': ARDUINO_MEGA.A11, ATMEGA128.51, JOYZXUNO_CFG.9
- new net JOYZXUNO_6': ARDUINO_MEGA.A12, ATMEGA128.50, JOYZXUNO_CFG.11
- new net JOYZXUNO_7': ARDUINO_MEGA.A13, ATMEGA128.49, JOYZXUNO_CFG.13
- new net JOYZXUNO_8': ARDUINO_MEGA.A14, ATMEGA128.48, JOYZXUNO_CFG.15
- new net JOYZXUNO_9': ARDUINO_MEGA.A15, ATMEGA128.47, JOYZXUNO_CFG.17
- new net KB_CONTROL: ARDUINO_MEGA.50, ATMEGA128.60, R7.1
- new net MISO1: SDCARD.7, SDCARD_ZXUNO.6
- new net MOSI1: SDCARD.2, SDCARD_ZXUNO.2
- new net N$5: KB_BIDIR.1, R7.2
- new net PW_CONTROL: ARDUINO_MEGA.51, ATMEGA128.44, PW_CONTROL.1
- new net RESET: ARDUINO_MEGA.53, ATMEGA128.46, EXTRASW_CFG.3, RESET_ZXUNO.2
- new net RST: ATMEGA128.20, ICSP.5
- new net SCK1: SDCARD.5, SDCARD_ZXUNO.5
- new net SWITCH: EXTRASW.3, EXTRASW.4, EXTRASW_CFG.2
- new net TEST: TAPE.1
- new net VDD1: SDCARD.4, SDCARD_ZXUNO.4
- net +5V: now also ARDUINO_MEGA.5V@1, ARDUINO_MEGA.5V@2, ATMEGA128.21, ATMEGA128.52, ATMEGA128.64, ICSP.2, JOYSTICK_1.5, TAPE.3, TZXDUINO.1, U$1.VCC, USB_ARDUINO.5, X5.1; no longer B1.5V@0, B1.5V@1, B1.5V@2, JOYSTICK1.5, PWCON_ZXUNO.1, TZXDUINO.8, U1.5V@1, U1.5V@2
- net AUDIO_L: now also INTERNAL_SPEAKERS.1, TAPE.2
- net AUDIO_R: now also INTERNAL_SPEAKERS.3
- net COMPOSITE: now also VIDEO_CFG.1; no longer JP3.1
- net CSYNC: now also VIDEO_CFG.3; no longer JP3.3
- net GND: now also INTERNAL_SPEAKERS.2, JOYSTICK_1.8, PW_CONTROL.2, PW_SWITCH.2, RESET_ZXUNO.1, SDCARD.3, SDCARD.6, SDCARD.M1, SDCARD.M2, SDCARD.M3, SDCARD.M4, SDCARD_ZXUNO.3, TAPE.5, TZXDUINO.2, TZXDUINO.9, X5.5, X5.6; no longer B1.GND@0, B1.GND@1, B1.GND@2, B1.GND@3, B1.GND@4, JOYSTICK1.8, PWCON_ZXUNO.2, TZXDUINO.7, U1.GND@0, U1.GND@1, U1.GND@4
- net IN_L: now also TAPE.4, TZXDUINO.8, X5.9
- net JOY2PS2_1: now also ARDUINO_MEGA.7, ATMEGA128.7, JOYSTICK_1.1; no longer B1.7, JOYSTICK1.1, U1.7
- net JOY2PS2_2: now also ARDUINO_MEGA.8, ATMEGA128.6, JOYSTICK_1.2; no longer B1.8, JOYSTICK1.2, U1.8
- net JOY2PS2_3: now also ARDUINO_MEGA.9, ATMEGA128.5, JOYSTICK_1.3; no longer B1.9, JOYSTICK1.3, U1.9
- net JOY2PS2_4: now also ARDUINO_MEGA.10, ATMEGA128.4, JOYSTICK_1.4; no longer B1.10, JOYSTICK1.4, U1.10
- net JOY2PS2_6: now also ARDUINO_MEGA.11, ATMEGA128.3, JOYSTICK_1.6; no longer B1.11, JOYSTICK1.6, U1.11
- net JOY2PS2_7: now also ARDUINO_MEGA.12, ATMEGA128.2, JOYSTICK_1.7; no longer B1.12, JOYSTICK1.7, U1.12
- net JOY2PS2_9: now also ARDUINO_MEGA.44, ATMEGA128.40, JOYSTICK_1.9; no longer B1.13, JOYSTICK1.9, U1.13
- net JOYZXUNO_1: now also JOYSTICK_2.1, JOYZXUNO_CFG.2; no longer JOYSTICK2.1
- net JOYZXUNO_2: now also JOYSTICK_2.2, JOYZXUNO_CFG.4; no longer JOYSTICK2.2
- net JOYZXUNO_3: now also JOYSTICK_2.3, JOYZXUNO_CFG.6; no longer JOYSTICK2.3
- net JOYZXUNO_4: now also JOYSTICK_2.4, JOYZXUNO_CFG.8; no longer JOYSTICK2.4
- net JOYZXUNO_5: now also JOYSTICK_2.5, JOYZXUNO_CFG.10; no longer JOYSTICK2.5
- net JOYZXUNO_6: now also JOYSTICK_2.6, JOYZXUNO_CFG.12; no longer JOYSTICK2.6
- net JOYZXUNO_7: now also JOYSTICK_2.7, JOYZXUNO_CFG.14; no longer JOYSTICK2.7
- net JOYZXUNO_8: now also JOYSTICK_2.8, JOYZXUNO_CFG.16; no longer JOYSTICK2.8
- net JOYZXUNO_9: now also JOYSTICK_2.9, JOYZXUNO_CFG.18; no longer JOYSTICK2.9
- net M1_KB1: now also ARDUINO_MEGA.23, ATMEGA128.14, KB1.1; no longer B1.23, JP2.1, U1.23
- net M1_KB10: now also ARDUINO_MEGA.41, ATMEGA128.37, KB1.10; no longer B1.41, JP2.10, U1.41
- net M1_KB11: now also ARDUINO_MEGA.43, ATMEGA128.39, KB1.11; no longer B1.43, JP2.11, U1.43
- net M1_KB12: now also ARDUINO_MEGA.45, ATMEGA128.41, KB1.12; no longer B1.45, JP2.12, U1.45
- net M1_KB13: now also ARDUINO_MEGA.47, ATMEGA128.42, KB1.13; no longer B1.47, JP2.13, U1.47
- net M1_KB2: now also ARDUINO_MEGA.25, ATMEGA128.16, KB1.2; no longer B1.25, JP2.2, U1.25
- net M1_KB3: now also ARDUINO_MEGA.27, ATMEGA128.18, KB1.3; no longer B1.27, JP2.3, U1.27
- net M1_KB4: now also ARDUINO_MEGA.29, ATMEGA128.25, KB1.4; no longer B1.29, JP2.4, U1.29
- net M1_KB5: now also ARDUINO_MEGA.31, ATMEGA128.27, KB1.5; no longer B1.31, JP2.5, U1.31
- net M1_KB6: now also ARDUINO_MEGA.33, ATMEGA128.29, KB1.6; no longer B1.33, JP2.6, U1.33
- net M1_KB7: now also ARDUINO_MEGA.35, ATMEGA128.31, KB1.7; no longer B1.35, JP2.7, U1.35
- net M1_KB8: now also ARDUINO_MEGA.37, ATMEGA128.33, KB1.8; no longer B1.37, JP2.8, U1.37
- net M1_KB9: now also ARDUINO_MEGA.39, ATMEGA128.35, KB1.9; no longer B1.39, JP2.9, U1.39
- net M2_KB1: now also ARDUINO_MEGA.22, ATMEGA128.13, ICSP.1, KB2.1; no longer B1.22, JP1.1, U1.22
- net M2_KB10: now also ARDUINO_MEGA.40, ATMEGA128.36, KB2.10; no longer B1.40, JP1.10, U1.40
- net M2_KB11: now also ARDUINO_MEGA.42, ATMEGA128.38, KB2.11; no longer B1.42, JP1.11, U1.42
- net M2_KB2: now also ARDUINO_MEGA.24, ATMEGA128.15, KB2.2; no longer B1.24, JP1.2, U1.24
- net M2_KB3: now also ARDUINO_MEGA.26, ATMEGA128.17, KB2.3; no longer B1.26, JP1.3, U1.26
- net M2_KB4: now also ARDUINO_MEGA.28, ATMEGA128.19, KB2.4; no longer B1.28, JP1.4, U1.28
- net M2_KB5: now also ARDUINO_MEGA.30, ATMEGA128.26, KB2.5; no longer B1.30, JP1.5, U1.30
- net M2_KB6: now also ARDUINO_MEGA.32, ATMEGA128.28, KB2.6; no longer B1.32, JP1.6, U1.32
- net M2_KB7: now also ARDUINO_MEGA.34, ATMEGA128.30, KB2.7; no longer B1.34, JP1.7, U1.34
- net M2_KB8: now also ARDUINO_MEGA.36, ATMEGA128.32, KB2.8; no longer B1.36, JP1.8, U1.36
- net M2_KB9: now also ARDUINO_MEGA.38, ATMEGA128.34, KB2.9; no longer B1.38, JP1.9, U1.38
- net N$1: now also VIDEO_CFG.2; no longer JP3.2
- net PS2_KBCLK: now also ARDUINO_MEGA.A2, ATMEGA128.59; no longer B1.A2, U1.A2
- net PS2_KBDATA: now also ARDUINO_MEGA.A3, ATMEGA128.58, KB_BIDIR.3; no longer B1.A3, U1.A3
- net PS2_KBDATA': now also KB_BIDIR.4
- net TZX_DOWN: now also ARDUINO_MEGA.4, ATMEGA128.10, TZXDUINO.5, X5.3; no longer B1.4, TZXDUINO.3, U1.4
- net TZX_PLAY: now also ARDUINO_MEGA.5, ATMEGA128.9, TZXDUINO.6, X5.8; no longer B1.5, TZXDUINO.4, U1.5
- net TZX_ROOT: now also ARDUINO_MEGA.2, ATMEGA128.12, ICSP.4, TZXDUINO.3, X5.2; no longer B1.2, TZXDUINO.1, U1.2
- net TZX_STOP: now also ARDUINO_MEGA.6, ATMEGA128.8, TZXDUINO.7, X5.4; no longer B1.6, TZXDUINO.5, U1.6
- net TZX_UP: now also ARDUINO_MEGA.3, ATMEGA128.11, ICSP.3, TZXDUINO.4, X5.7; no longer B1.3, TZXDUINO.2, U1.3
Other:
- board text added: "+5V"
- board text added: "1"
- board text added: "2"
- board text added: "3"
- board text added: "4"
- board text added: "5"
- board text added: "6"
- board text added: "7"
- board text added: "8"
- board text added: "9"
- board text added: "AUDIO_L"
- board text added: "AUDIO_R"
- board text added: "CS1"
- board text added: "D+"
- board text added: "D-"
- board text added: "DOWN"
- board text added: "FIRE 1"
- board text added: "FIRE 2"
- board text added: "FIRE 3 / VCC"
- board text added: "GND"
- board text added: "ID"
- board text added: "LEFT"
- board text added: "MISO"
- board text added: "MOSI"
- board text added: "RIGHT"
- board text added: "SCK1"
- board text added: "UP"
- board text added: "VCC / FIRE 3"
- board text added: "VDD1"

Commit message: Update 3
Parts:
- removed JOYSTICK_ZXUNO: (no value), SparkFun-Connectors:DB9
- removed JOYZXUNO_CFG: (no value), pinhead:2X09
- added JOY: DB9_FEMALE, SparkFun-Connectors:DB9
- added LED: 22-23-2021, con-molex:22-23-2021
- added RECOVERY, TAPE_CFG1, TAPE_CFG2: (no value), pinhead:2X03
- added Y1: 16MHz, Cristalli:RESONATOR
- moved INTERNAL_SPEAKERS 127.6 mm to (-27.8, -53.0), turned to 90 degrees
- moved Q4 95.9 mm to (-16.3, 48.7)
- moved RGBAUDIO_ZXUNO 82.5 mm to (7.67, 37.3)
- moved X2 82.2 mm to (-16.5, -40.0), turned to 270 degrees
- moved C3 75.9 mm to (3.46, 63.0)
- moved Q3 75.9 mm to (3.46, 56.5)
- moved R5 75.9 mm to (-3.64, 57.7)
- moved R6 75.9 mm to (10.1, 57.7)
- moved RGBAUDIO_ZXUNO' 66.7 mm to (28.2, 68.2)
- moved ICSP 66.6 mm to (-27.8, -35.8)
- moved Q1 47.2 mm to (-36.6, 56.4)
- moved R2 47.2 mm to (-43.8, 58.4)
- moved R3 47.2 mm to (-23.4, 57.7)
- moved R4 47.2 mm to (-9.34, 57.6)
- moved C1 47.2 mm to (-36.5, 63.2)
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Connections:
- net PS2_MSDAT renamed PS2_MSDATA
- removed net JOYZXUNO_1': ARDUINO_MEGA.A7, ATMEGA128.57, JOYZXUNO_CFG.1
- removed net JOYZXUNO_2': ARDUINO_MEGA.A8, ATMEGA128.56, JOYZXUNO_CFG.3
- removed net JOYZXUNO_3': ARDUINO_MEGA.A9, ATMEGA128.55, JOYZXUNO_CFG.5
- removed net JOYZXUNO_4': ARDUINO_MEGA.A10, ATMEGA128.54, JOYZXUNO_CFG.7
- removed net JOYZXUNO_5': ARDUINO_MEGA.A11, ATMEGA128.51, JOYZXUNO_CFG.9
- removed net JOYZXUNO_6': ARDUINO_MEGA.A12, ATMEGA128.50, JOYZXUNO_CFG.11
- removed net JOYZXUNO_7': ARDUINO_MEGA.A13, ATMEGA128.49, JOYZXUNO_CFG.13
- removed net JOYZXUNO_8': ARDUINO_MEGA.A14, ATMEGA128.48, JOYZXUNO_CFG.15
- removed net JOYZXUNO_9': ARDUINO_MEGA.A15, ATMEGA128.47, JOYZXUNO_CFG.17
- removed net PS2_KBDAT: PS/2_ZXUNO'.1, PS/2_ZXUNO.1
- removed net TEST: TAPE.1
- new net N$6: ATMEGA128.23, Y1.3
- new net N$7: ATMEGA128.24, Y1.1
- new net N/C: TAPE_CFG2.1, TAPE_CFG2.2
- new net PW_LED: ARDUINO_MEGA.49, ATMEGA128.47, LED.1
- new net TAPE_1: TAPE.1, TAPE_CFG2.3
- new net TAPE_2: TAPE.2, TAPE_CFG1.3
- new net TAPE_4: TAPE.4, TAPE_CFG1.4
- new net TAPE_5: TAPE.5, TAPE_CFG2.4
- net +5V: now also JOYSTICK_1.14
- net AUDIO_L: now also TAPE_CFG1.1, TAPE_CFG1.2; no longer TAPE.2
- net GND: now also JOYSTICK_1.17, LED.2, RECOVERY.3, RECOVERY.4, TAPE_CFG2.5, TAPE_CFG2.6, X4.SH1, X4.SH2, X4.SH3; no longer TAPE.5
- net GND_POW: now also R7.1, Y1.2; no longer KB_BIDIR.2
- net IN_L: now also TAPE_CFG1.5, TAPE_CFG1.6; no longer TAPE.4
- net JOY2PS2_1: now also JOYSTICK_1.10
- net JOY2PS2_2: now also JOYSTICK_1.11
- net JOY2PS2_3: now also JOYSTICK_1.12
- net JOY2PS2_4: now also JOYSTICK_1.13
- net JOY2PS2_6: now also JOYSTICK_1.15
- net JOY2PS2_7: now also JOYSTICK_1.16
- net JOY2PS2_9: now also JOYSTICK_1.18
- net JOYZXUNO_1: now also JOY.1, JOYSTICK_2.10; no longer JOYSTICK_ZXUNO.1, JOYZXUNO_CFG.2
- net JOYZXUNO_2: now also JOY.2, JOYSTICK_2.11, RECOVERY.1; no longer JOYSTICK_ZXUNO.2, JOYZXUNO_CFG.4
- net JOYZXUNO_3: now also JOY.3, JOYSTICK_2.12; no longer JOYSTICK_ZXUNO.3, JOYZXUNO_CFG.6
- net JOYZXUNO_4: now also JOY.4, JOYSTICK_2.13; no longer JOYSTICK_ZXUNO.4, JOYZXUNO_CFG.8
- net JOYZXUNO_5: now also JOY.5, JOYSTICK_2.14; no longer JOYSTICK_ZXUNO.5, JOYZXUNO_CFG.10
- net JOYZXUNO_6: now also JOY.6, JOYSTICK_2.15, RECOVERY.2; no longer JOYSTICK_ZXUNO.6, JOYZXUNO_CFG.12
- net JOYZXUNO_7: now also JOY.7, JOYSTICK_2.16; no longer JOYSTICK_ZXUNO.7, JOYZXUNO_CFG.14
- net JOYZXUNO_8: now also JOY.8, JOYSTICK_2.17; no longer JOYSTICK_ZXUNO.8, JOYZXUNO_CFG.16
- net JOYZXUNO_9: now also JOY.9, JOYSTICK_2.18; no longer JOYSTICK_ZXUNO.9, JOYZXUNO_CFG.18
- net KB_CONTROL: now also KB_BIDIR.1; no longer R7.1
- net N$5: now also KB_BIDIR.2; no longer KB_BIDIR.1
- net PE1: no longer X4.SH1
- net PE2: no longer X4.SH2
- net PE3: no longer X4.SH3
- net PS2_KBDATA: now also PS/2_ZXUNO'.1, PS/2_ZXUNO.1
Other:
- outline, holes or cut-outs redrawn
- board text added: "+3.3V"
- board text added: "B"
- board text added: "G"
- board text added: "HSYNC"
- board text added: "OFF"
- board text added: "ON"
- board text added: "R"
- board text added: "VSYNC"
- board text removed: "6"
- board text removed: "7"
- board text removed: "8"
- board text removed: "9"
- board text removed: "DOWN"
- board text removed: "FIRE 1"
- board text removed: "FIRE 2"
- board text removed: "FIRE 3 / VCC"
- board text removed: "LEFT"
- board text removed: "RIGHT"
- board text removed: "UP"
- board text removed: "VCC / FIRE 3"
