File: ZXUnoCompanion-2/ZXUno_Companion_2.sch (EAGLE design)
At the start: 44 parts, among them Q1 2N3904, Q2 2N3904, Q3 2N3904, Q4 2N3904, U1 ARDUINO_MEGA_R3FULL, X1 TOBU3, X2 TOBU3, X3 DB15

Commit message: Update 2
Parts:
- removed B1: MEGA2560_COREFULL, spark2k06:MEGA2560_COREFULL
- removed JP1: (no value), pinhead:PINHD-1X11
- removed JP2: (no value), pinhead:PINHD-1X13
- removed PWCON_ZXUNO: (no value), pinhead:PINHD-1X4
- removed U1: ARDUINO_MEGA_R3FULL, SparkFun-Boards:ARDUINO_MEGA_R3FULL
- added ARDUINO_MEGA: ARDUINO_MEGA_R3FULL, SparkFun-Boards2:ARDUINO_MEGA_R3FULL
- added ATMEGA128: MEGA128-A, atmel:MEGA128-A
- added EXTRASW: PS-22F03, A03 PS-22F03:PS-22F03
- added EXTRASW_CFG, INTERNAL_SPEAKERS: (no value), pinhead:PINHD-1X3
- added ICSP: AVR_SPI_PRG_6NS, SparkFun-Connectors:AVR_SPI_PRG_6NS
- added JOYZXUNO_CFG: (no value), pinhead:PINHD-2X9
- added KB1: (no value), pinhead:PINHD-1X13
- added KB2: (no value), pinhead:PINHD-1X11
- added KB_BIDIR: PC817, optocoupler:PC817
- added PW_CONTROL: IRLML6344TRPBF, International_Rectifier_By_element14_Batch_1:IRLML6344TRPBF
- added PW_SWITCH: (no value), pinhead:PINHD-1X2
- added R7: 220R, resistor:R-EU_0204/7
- added SDCARD: (no value), zxuno_rev_mcleod:SDCARD
- added SDCARD_ZXUNO: (no value), pinhead:PINHD-1X6
- added TAPE: 22-23-2051, con-molex:22-23-2051
- added U$1: MICRO-USB-B, micro usb B - 4LEGS:MICRO-USB-B
- added USB_ARDUINO: (no value), pinhead:PINHD-1X5
- added X5: (no value), con-subd-spark2k06:F09D
- R1, R2, R3, R4, R5, R6: device resistor:R-EU_0207/10 -> resistor:R-EU_0204/7
- TZXDUINO: device pinhead:PINHD-2X4 -> pinhead:PINHD-2X5
- renumbered JOYSTICK1 to JOYSTICK_1, JOYSTICK2 to JOYSTICK_2, JP3 to VIDEO_CFG
Connections:
- removed net SW1: PWCON_ZXUNO.3
- removed net SW2: PWCON_ZXUNO.4
- new net CS1: SDCARD.CD/DAT3/CS, SDCARD_ZXUNO.1
- new net D+: U$1.D+, USB_ARDUINO.3
- new net D-: U$1.D-, USB_ARDUINO.4
- new net EXTRA: ARDUINO_MEGA.52, ATMEGA128.(AD6)PA6, EXTRASW_CFG.1
- new net GND_POW: ARDUINO_MEGA.GND@0, ARDUINO_MEGA.GND@1, ARDUINO_MEGA.GND@4, ATMEGA128.GND, ATMEGA128.GND@1, ATMEGA128.GND@2, EXTRASW.5, EXTRASW.6, ICSP.6, KB_BIDIR.C, PW_CONTROL.D, PW_SWITCH.1, U$1.GND, USB_ARDUINO.1
- new net ID: U$1.ID, USB_ARDUINO.2
- new net JOYZXUNO_1': ARDUINO_MEGA.A7, ATMEGA128.PF4(ADC4/TCK), JOYZXUNO_CFG.1
- new net JOYZXUNO_2': ARDUINO_MEGA.A8, ATMEGA128.PF5(ADC5/TMS), JOYZXUNO_CFG.3
- new net JOYZXUNO_3': ARDUINO_MEGA.A9, ATMEGA128.PF6(ADC6/TDO), JOYZXUNO_CFG.5
- new net JOYZXUNO_4': ARDUINO_MEGA.A10, ATMEGA128.PF7(ADC7/TDI), JOYZXUNO_CFG.7
- new net JOYZXUNO_5': ARDUINO_MEGA.A11, ATMEGA128.(AD0)PA0, JOYZXUNO_CFG.9
- new net JOYZXUNO_6': ARDUINO_MEGA.A12, ATMEGA128.(AD1)PA1, JOYZXUNO_CFG.11
- new net JOYZXUNO_7': ARDUINO_MEGA.A13, ATMEGA128.(AD2)PA2, JOYZXUNO_CFG.13
- new net JOYZXUNO_8': ARDUINO_MEGA.A14, ATMEGA128.(AD3)PA3, JOYZXUNO_CFG.15
- new net JOYZXUNO_9': ARDUINO_MEGA.A15, ATMEGA128.(AD4)PA4, JOYZXUNO_CFG.17
- new net KB_CONTROL: ARDUINO_MEGA.50, ATMEGA128.PF1(ADC1), R7.1
- new net MISO1: SDCARD.DAT0/DO, SDCARD_ZXUNO.6
- new net MOSI1: SDCARD.CMD/DI, SDCARD_ZXUNO.2
- new net N$5: KB_BIDIR.A, R7.2
- new net PW_CONTROL: ARDUINO_MEGA.51, ATMEGA128.(AD7)PA7, PW_CONTROL.G
- new net RESET: ARDUINO_MEGA.53, ATMEGA128.(AD5)PA5, EXTRASW_CFG.3, RESET_ZXUNO.2
- new net RST: ATMEGA128.RESET, ICSP.5
- new net SCK1: SDCARD.CLK/SCLK, SDCARD_ZXUNO.5
- new net SWITCH: EXTRASW.3, EXTRASW.4, EXTRASW_CFG.2
- new net TEST: TAPE-1.S
- new net VDD1: SDCARD.VDD, SDCARD_ZXUNO.4
- net +5V: now also ARDUINO_MEGA.5V@1, ARDUINO_MEGA.5V@2, ATMEGA128.AVCC, ATMEGA128.VCC, ATMEGA128.VCC@1, ICSP.2, TAPE-3.S, TZXDUINO.1, U$1.VCC, USB_ARDUINO.5, X5.1; no longer B1.5V@0, B1.5V@1, B1.5V@2, PWCON_ZXUNO.1, TZXDUINO.8, U1.5V@1, U1.5V@2
- net AUDIO_L: now also INTERNAL_SPEAKERS.1, TAPE-2.S
- net AUDIO_R: now also INTERNAL_SPEAKERS.3
- net GND: now also INTERNAL_SPEAKERS.2, PW_CONTROL.S, PW_SWITCH.2, RESET_ZXUNO.1, SDCARD.GND@1, SDCARD.GND@2, SDCARD.GND@3, SDCARD.GND@4, SDCARD.VSS1, SDCARD.VSS2, SDCARD_ZXUNO.3, TAPE-5.S, TZXDUINO.2, TZXDUINO.9, X5.5, X5.6; no longer B1.GND@0, B1.GND@1, B1.GND@2, B1.GND@3, B1.GND@4, PWCON_ZXUNO.2, TZXDUINO.7, U1.GND@0, U1.GND@1, U1.GND@4
- net IN_L: now also TAPE-4.S, TZXDUINO.8, X5.9
- net JOY2PS2_1: now also ARDUINO_MEGA.7, ATMEGA128.(OC3C/INT5)PE5; no longer B1.7, U1.7
- net JOY2PS2_2: now also ARDUINO_MEGA.8, ATMEGA128.(OC3B/INT4)PE4; no longer B1.8, U1.8
- net JOY2PS2_3: now also ARDUINO_MEGA.9, ATMEGA128.(OC3A/AIN1)PE3; no longer B1.9, U1.9
- net JOY2PS2_4: now also ARDUINO_MEGA.10, ATMEGA128.(XCK0/AIN0)PE2; no longer B1.10, U1.10
- net JOY2PS2_6: now also ARDUINO_MEGA.11, ATMEGA128.(TXD/PDO)PE1; no longer B1.11, U1.11
- net JOY2PS2_7: now also ARDUINO_MEGA.12, ATMEGA128.(RXD/PDI)PE0; no longer B1.12, U1.12
- net JOY2PS2_9: now also ARDUINO_MEGA.44, ATMEGA128.(A13)PC5; no longer B1.13, U1.13
- net JOYZXUNO_1: now also JOYZXUNO_CFG.2
- net JOYZXUNO_2: now also JOYZXUNO_CFG.4
- net JOYZXUNO_3: now also JOYZXUNO_CFG.6
- net JOYZXUNO_4: now also JOYZXUNO_CFG.8
- net JOYZXUNO_5: now also JOYZXUNO_CFG.10
- net JOYZXUNO_6: now also JOYZXUNO_CFG.12
- net JOYZXUNO_7: now also JOYZXUNO_CFG.14
- net JOYZXUNO_8: now also JOYZXUNO_CFG.16
- net JOYZXUNO_9: now also JOYZXUNO_CFG.18
- net M1_KB1: now also ARDUINO_MEGA.23, ATMEGA128.(OC0)PB4, KB1.1; no longer B1.23, JP2.1, U1.23
- net M1_KB10: now also ARDUINO_MEGA.41, ATMEGA128.(A10)PC2, KB1.10; no longer B1.41, JP2.10, U1.41
- net M1_KB11: now also ARDUINO_MEGA.43, ATMEGA128.(A12)PC4, KB1.11; no longer B1.43, JP2.11, U1.43
- net M1_KB12: now also ARDUINO_MEGA.45, ATMEGA128.(A14)PC6, KB1.12; no longer B1.45, JP2.12, U1.45
- net M1_KB13: now also ARDUINO_MEGA.47, ATMEGA128.(A15)PC7, KB1.13; no longer B1.47, JP2.13, U1.47
- net M1_KB2: now also ARDUINO_MEGA.25, ATMEGA128.(OC1B)PB6, KB1.2; no longer B1.25, JP2.2, U1.25
- net M1_KB3: now also ARDUINO_MEGA.27, ATMEGA128.PG3(TOSC2), KB1.3; no longer B1.27, JP2.3, U1.27
- net M1_KB4: now also ARDUINO_MEGA.29, ATMEGA128.(SCL/INT0)PD0, KB1.4; no longer B1.29, JP2.4, U1.29
- net M1_KB5: now also ARDUINO_MEGA.31, ATMEGA128.(RXD1/INT2)PD2, KB1.5; no longer B1.31, JP2.5, U1.31
- net M1_KB6: now also ARDUINO_MEGA.33, ATMEGA128.(IC1)PD4, KB1.6; no longer B1.33, JP2.6, U1.33
- net M1_KB7: now also ARDUINO_MEGA.35, ATMEGA128.(T1)PD6, KB1.7; no longer B1.35, JP2.7, U1.35
- net M1_KB8: now also ARDUINO_MEGA.37, ATMEGA128.PG0(WR), KB1.8; no longer B1.37, JP2.8, U1.37
- net M1_KB9: now also ARDUINO_MEGA.39, ATMEGA128.(A8)PC0, KB1.9; no longer B1.39, JP2.9, U1.39
- net M2_KB1: now also ARDUINO_MEGA.22, ATMEGA128.(MISO)PB3, ICSP.1, KB2.1; no longer B1.22, JP1.1, U1.22
- net M2_KB10: now also ARDUINO_MEGA.40, ATMEGA128.(A9)PC1, KB2.10; no longer B1.40, JP1.10, U1.40
- net M2_KB11: now also ARDUINO_MEGA.42, ATMEGA128.(A11)PC3, KB2.11; no longer B1.42, JP1.11, U1.42
- net M2_KB2: now also ARDUINO_MEGA.24, ATMEGA128.(OC1A)PB5, KB2.2; no longer B1.24, JP1.2, U1.24
- net M2_KB3: now also ARDUINO_MEGA.26, ATMEGA128.(OC2/OC1C)PB7, KB2.3; no longer B1.26, JP1.3, U1.26
- net M2_KB4: now also ARDUINO_MEGA.28, ATMEGA128.PG4(TOSC1), KB2.4; no longer B1.28, JP1.4, U1.28
- net M2_KB5: now also ARDUINO_MEGA.30, ATMEGA128.(SDA/INT1)PD1, KB2.5; no longer B1.30, JP1.5, U1.30
- net M2_KB6: now also ARDUINO_MEGA.32, ATMEGA128.(TXD1/INT3)PD3, KB2.6; no longer B1.32, JP1.6, U1.32
- net M2_KB7: now also ARDUINO_MEGA.34, ATMEGA128.(XCK1)PD5, KB2.7; no longer B1.34, JP1.7, U1.34
- net M2_KB8: now also ARDUINO_MEGA.36, ATMEGA128.(T2)PD7, KB2.8; no longer B1.36, JP1.8, U1.36
- net M2_KB9: now also ARDUINO_MEGA.38, ATMEGA128.PG1(RD), KB2.9; no longer B1.38, JP1.9, U1.38
- net PS2_KBCLK: now also ARDUINO_MEGA.A2, ATMEGA128.PF2(ADC2); no longer B1.A2, U1.A2
- net PS2_KBDATA: now also ARDUINO_MEGA.A3, ATMEGA128.PF3(ADC3), KB_BIDIR.EMIT; no longer B1.A3, U1.A3
- net PS2_KBDATA': now also KB_BIDIR.COL
- net TZX_DOWN: now also ARDUINO_MEGA.4, ATMEGA128.(SS)PB0, TZXDUINO.5, X5.3; no longer B1.4, TZXDUINO.3, U1.4
- net TZX_PLAY: now also ARDUINO_MEGA.5, ATMEGA128.(IC3/INT7)PE7, TZXDUINO.6, X5.8; no longer B1.5, TZXDUINO.4, U1.5
- net TZX_ROOT: now also ARDUINO_MEGA.2, ATMEGA128.(MOSI)PB2, ICSP.4, TZXDUINO.3, X5.2; no longer B1.2, TZXDUINO.1, U1.2
- net TZX_STOP: now also ARDUINO_MEGA.6, ATMEGA128.(T3/INT6)PE6, TZXDUINO.7, X5.4; no longer B1.6, TZXDUINO.5, U1.6
- net TZX_UP: now also ARDUINO_MEGA.3, ATMEGA128.(SCK)PB1, ICSP.3, TZXDUINO.4, X5.7; no longer B1.3, TZXDUINO.2, U1.3
Other:
- moved on the sheet: AUDIO_EXTERNAL, EAR_ZXUNO, EXTERNAL_ZXUNO, PS/2_EXTERNAL, PS/2_ZXUNO, PS/2_ZXUNO', RESET_ZXUNO, RGBAUDIO_ZXUNO', RGBAUDIO_ZXUNO-1, RGBAUDIO_ZXUNO-2, RGBAUDIO_ZXUNO-3, RGBAUDIO_ZXUNO-4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

Commit message: Update 3
Parts:
- removed JOYSTICK_ZXUNO: (no value), SparkFun-Connectors:DB9FEMALE
- removed JOYZXUNO_CFG: (no value), pinhead:PINHD-2X9
- added JOY: DB9_FEMALE, SparkFun-Connectors:DB9_FEMALE
- added LED: 22-23-2021, con-molex:22-23-2021
- added RECOVERY, TAPE_CFG1, TAPE_CFG2: (no value), pinhead:PINHD-2X3
- added Y1: 16MHz, Cristalli:0011_CSTCE16M0V53-R0
Connections:
- net PS2_MSDAT renamed PS2_MSDATA
- removed net JOYZXUNO_1': ARDUINO_MEGA.A7, ATMEGA128.PF4(ADC4/TCK), JOYZXUNO_CFG.1
- removed net JOYZXUNO_2': ARDUINO_MEGA.A8, ATMEGA128.PF5(ADC5/TMS), JOYZXUNO_CFG.3
- removed net JOYZXUNO_3': ARDUINO_MEGA.A9, ATMEGA128.PF6(ADC6/TDO), JOYZXUNO_CFG.5
- removed net JOYZXUNO_4': ARDUINO_MEGA.A10, ATMEGA128.PF7(ADC7/TDI), JOYZXUNO_CFG.7
- removed net JOYZXUNO_5': ARDUINO_MEGA.A11, ATMEGA128.(AD0)PA0, JOYZXUNO_CFG.9
- removed net JOYZXUNO_6': ARDUINO_MEGA.A12, ATMEGA128.(AD1)PA1, JOYZXUNO_CFG.11
- removed net JOYZXUNO_7': ARDUINO_MEGA.A13, ATMEGA128.(AD2)PA2, JOYZXUNO_CFG.13
- removed net JOYZXUNO_8': ARDUINO_MEGA.A14, ATMEGA128.(AD3)PA3, JOYZXUNO_CFG.15
- removed net JOYZXUNO_9': ARDUINO_MEGA.A15, ATMEGA128.(AD4)PA4, JOYZXUNO_CFG.17
- removed net PS2_KBDAT: PS/2_ZXUNO'.1, PS/2_ZXUNO.1
- removed net TEST: TAPE-1.S
- new net N$6: ATMEGA128.XTAL2, Y1.3
- new net N$7: ATMEGA128.XTAL1, Y1.1
- new net N/C: TAPE_CFG2.1, TAPE_CFG2.2
- new net PW_LED: ARDUINO_MEGA.49, ATMEGA128.(AD4)PA4, LED-1.S
- new net TAPE_1: TAPE-1.S, TAPE_CFG2.3
- new net TAPE_2: TAPE-2.S, TAPE_CFG1.3
- new net TAPE_4: TAPE-4.S, TAPE_CFG1.4
- new net TAPE_5: TAPE-5.S, TAPE_CFG2.4
- net +5V: now also JOYSTICK_1.14
- net AUDIO_L: now also TAPE_CFG1.1, TAPE_CFG1.2; no longer TAPE-2.S
- net GND: now also JOYSTICK_1.17, LED-2.S, RECOVERY.3, RECOVERY.4, TAPE_CFG2.5, TAPE_CFG2.6, X4.PE1, X4.PE2, X4.PE3; no longer TAPE-5.S
- net GND_POW: now also R7.1, Y1.2; no longer KB_BIDIR.C
- net IN_L: now also TAPE_CFG1.5, TAPE_CFG1.6; no longer TAPE-4.S
- net JOY2PS2_1: now also JOYSTICK_1.10
- net JOY2PS2_2: now also JOYSTICK_1.11
- net JOY2PS2_3: now also JOYSTICK_1.12
- net JOY2PS2_4: now also JOYSTICK_1.13
- net JOY2PS2_6: now also JOYSTICK_1.15
- net JOY2PS2_7: now also JOYSTICK_1.16
- net JOY2PS2_9: now also JOYSTICK_1.18
- net JOYZXUNO_1: now also JOY.1, JOYSTICK_2.10; no longer JOYSTICK_ZXUNO.1, JOYZXUNO_CFG.2
- net JOYZXUNO_2: now also JOY.2, JOYSTICK_2.11, RECOVERY.1; no longer JOYSTICK_ZXUNO.2, JOYZXUNO_CFG.4
- net JOYZXUNO_3: now also JOY.3, JOYSTICK_2.12; no longer JOYSTICK_ZXUNO.3, JOYZXUNO_CFG.6
- net JOYZXUNO_4: now also JOY.4, JOYSTICK_2.13; no longer JOYSTICK_ZXUNO.4, JOYZXUNO_CFG.8
- net JOYZXUNO_5: now also JOY.5, JOYSTICK_2.14; no longer JOYSTICK_ZXUNO.5, JOYZXUNO_CFG.10
- net JOYZXUNO_6: now also JOY.6, JOYSTICK_2.15, RECOVERY.2; no longer JOYSTICK_ZXUNO.6, JOYZXUNO_CFG.12
- net JOYZXUNO_7: now also JOY.7, JOYSTICK_2.16; no longer JOYSTICK_ZXUNO.7, JOYZXUNO_CFG.14
- net JOYZXUNO_8: now also JOY.8, JOYSTICK_2.17; no longer JOYSTICK_ZXUNO.8, JOYZXUNO_CFG.16
- net JOYZXUNO_9: now also JOY.9, JOYSTICK_2.18; no longer JOYSTICK_ZXUNO.9, JOYZXUNO_CFG.18
- net KB_CONTROL: now also KB_BIDIR.A; no longer R7.1
- net N$5: now also KB_BIDIR.C; no longer KB_BIDIR.A
- net PS2_KBDATA: now also PS/2_ZXUNO'.1, PS/2_ZXUNO.1
Other:
- moved on the sheet: EXTRASW, JOYSTICK_ZXUNO_BIS, R7, RGBAUDIO_ZXUNO-1, RGBAUDIO_ZXUNO-2, RGBAUDIO_ZXUNO-3, RGBAUDIO_ZXUNO-4, RGBAUDIO_ZXUNO-5, RGBAUDIO_ZXUNO-6, RGBAUDIO_ZXUNO-7, RGBAUDIO_ZXUNO-8, RGBAUDIO_ZXUNO-9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
